File: small-display/small-display.kicad_sch (KiCad schematic)
At the start: 30 parts, among them J1 USB_C_Receptacle_USB2.0, J2 Micro_SD_Card_Det, J5 F32D-1A7Y1-21040, U1 TPD4EUSB30, U2 74LVC1G07SE-7, U3 RT9742GGJ5, U4 PAM2804AAB010, U5 USB2412-DZK, Y1 ECS-240-8-33-AGN-TR

Commit message: Minor changes.
Connections:
- net !RESET renamed GPIO_27_!RESET
- net !WRITE renamed GPIO_07_!WRITE
- net DAT_CMD renamed GPIO_26_DAT_CMD
- net DB0 renamed GPIO_08_DB0
- net DB1 renamed GPIO_09_DB1
- net DB10 renamed GPIO_18_DB10
- net DB11 renamed GPIO_19_DB11
- net DB12 renamed GPIO_20_DB12
- net DB13 renamed GPIO_21_DB13
- net DB14 renamed GPIO_22_DB14
- net DB15 renamed GPIO_23_DB15
- net DB2 renamed GPIO_10_DB2
- net DB3 renamed GPIO_11_DB3
- net DB4 renamed GPIO_12_DB4
- net DB5 renamed GPIO_13_DB5
- net DB6 renamed GPIO_14_DB6
- net DB7 renamed GPIO_15_DB7
- net DB8 renamed GPIO_16_DB8
- net DB9 renamed GPIO_17_DB9
- net PWM renamed GPIO_02_PWM
- no-connect marks 20 -> 28
Other:
- note added: "LCD panel connections"
- note added: "SCHEMATIC TODO: [x] Choose xtal for USB hub [x] Choose caps for xtal [x] Wire up USB hub (both ends) [x] Decide on RESET line for USB hub [x] Wire up power connections [x] Figure out GPIO mappings for display [ ] Choose a GPIO for USB_RESET [ ] Wire up display connections [ ] Review all RPi pinouts vs. CM4IO"
- note removed: "SCHEMATIC TODO: [x] Choose xtal for USB hub [x] Choose caps for xtal [x] Wire up USB hub (both ends) [x] Decide on RESET line for USB hub [x] Wire up power connections [ ] Figure out GPIO mappings for display [ ] Choose a GPIO for USB_RESET [ ] Wire up display connections"
- moved on the sheet: C2, C3, J5, L1, R4, R5, U4

Commit message: Continued work on small display PCB.
Parts:
- added TP1, TP2, TP3, TP4, TP5, TP6, TP7, TP8: TestPoint, TestPoint:TestPoint_Pad_D1.0mm, symbol Connector:TestPoint
- C4, C5: renamed from C?; footprint (none) -> Capacitor_SMD:C_0603_1608Metric
- R4, R5, R6, R7, R8: footprint Resistor_SMD:R_0603_1608Metric -> Resistor_SMD:R_0402_1005Metric
- R9: renamed from R?; footprint (none) -> Resistor_SMD:R_0402_1005Metric
- gave numbers to parts that had none: 1
Connections:
- net +5V: now also TP3.1
- net LED_A: now also TP7.1
- net LED_K: now also TP8.1
- net SD_PWR: now also TP1.1
- net SD_PWR_ON: now also TP5.1
- net at U5.17 (~{RESET_IN}), U6.4 (Y): now also TP6.1
- net GPIO_02_PWM renamed GPIO_25_PWM
- net GPIO_25_PWM: now also TP2.1
- net USB_RESET renamed GPIO_02_USB_!RESET
- net GPIO_02_USB_!RESET: now also TP4.1
Other:
- note added: "From the PAM2804 data sheet: I_{LED} = 0.1 V / R_{S} ∴ R_{S} = 0.1 V / I_{LED} From the NHD-2.4-240320CF-CSXN#-F data sheet: I_{LED} = 100 mA Therefore: R_{S} = 0.1 V / 0.1 A = 1 Ω In our circuit, R_{S} is part R5."
- note added: "GPIO_02_USB_!RESET is mapped to an RPi GPIO that is pulled high by default, so the system boots up with USB enabled."
- note added: "GPIO_25_PWM is mapped to an RPi GPIO that is pulled low by default. This ensures that the system turns on with the screen dark, until it is illuminated by software. This prevents the screen from "flashing" at full brightness momentarily when powered up, and potentially ruining the viewer's night vision!"
- note added: "SCHEMATIC TODO: [x] Choose xtal for USB hub [x] Choose caps for xtal [x] Wire up USB hub (both ends) [x] Decide on RESET line for USB hub [x] Wire up power connections [x] Figure out GPIO mappings for display [x] Choose a GPIO for USB_RESET [ ] Wire up display connections [ ] Review all RPi pinouts vs. CM4IO"
- note removed: "From the PAM2804 data sheet: I_{LED} = 0.1 V / R_{S} ∴ R_{S} = 0.1 V / I_{LED} From the NHD-2.4-240320CF-CSXN#-F data sheet: I_{LED} = 100 mA Therefore R_{S} = 0.1 V / 0.1 A = 1 Ω"
- note removed: "SCHEMATIC TODO: [x] Choose xtal for USB hub [x] Choose caps for xtal [x] Wire up USB hub (both ends) [x] Decide on RESET line for USB hub [x] Wire up power connections [x] Figure out GPIO mappings for display [ ] Choose a GPIO for USB_RESET [ ] Wire up display connections [ ] Review all RPi pinouts vs. CM4IO"
- note removed: "USB_RESET is mapped to an RPi GPIO that is pulled high by default."
- moved on the sheet: C2, C3, J5, L1, R3, R4, R5, U3, U4

Commit message: More work on small display.
Parts:
- removed J1: USB_C_Receptacle_USB2.0, CM4IO:USB411503C, symbol Connector:USB_C_Receptacle_USB2.0
- added J1: 2047110001, airball-hardware:MOLEX_2047110001, symbol airball-hardware:2047110001
- added TP10, TP11, TP12, TP9: TestPoint, TestPoint:TestPoint_Pad_D1.0mm, symbol Connector:TestPoint
Connections:
- net +5V: now also J1.A4 (VBUS_A), J1.A9 (VBUS_A), J1.B4 (VBUS_B), J1.B9 (VBUS_B)
- net GND: now also J1.A1 (GND_A), J1.A12 (GND_A), J1.B1 (GND_B), J1.B12 (GND_B), J1.S1 (SHIELD), J1.S2 (SHIELD), J1.S3 (SHIELD), J1.S4 (SHIELD), J1.S5 (SHIELD), J1.S6 (SHIELD)
- net USB2_N: now also TP9.1
- net USB2_P: now also TP10.1
- net USBD_N: now also J1.A7 (D1-), J1.B7 (D2-), TP11.1
- net USBD_P: now also J1.A6 (D1+), J1.B6 (D2+), TP12.1
- net at R7.2: now also J1.A5 (CC1)
- net at R6.2: now also J1.B5 (CC2)
- no-connect marks 28 -> 36
Other:
- note added: "R6 & R7 request USB-PD 5V 3A."
- note added: "SCHEMATIC TODO: [x] Choose xtal for USB hub [x] Choose caps for xtal [x] Wire up USB hub (both ends) [x] Decide on RESET line for USB hub [x] Wire up power connections [x] Figure out GPIO mappings for display [x] Choose a GPIO for USB_RESET [ ] Wire up display connections [ ] Review all RPi pinouts vs. CM4IO [x] Figure out J1 footprint & pinouts"
- note removed: "Request USB-PD 5V 3A power"
- note removed: "SCHEMATIC TODO: [x] Choose xtal for USB hub [x] Choose caps for xtal [x] Wire up USB hub (both ends) [x] Decide on RESET line for USB hub [x] Wire up power connections [x] Figure out GPIO mappings for display [x] Choose a GPIO for USB_RESET [ ] Wire up display connections [ ] Review all RPi pinouts vs. CM4IO"
- moved on the sheet: R6, R7, TP3, TP4, TP6, U1, U6

Commit message: More routing and design of small display.
Parts:
- added C6: 0.1uF, Capacitor_SMD:C_0603_1608Metric, symbol Device:C
- added U7: M24M01-DFDW6TP, airball-hardware:TSSOP_FDW6TP_STM, symbol airball-hardware:M24M01-DFDW6TP
Connections:
- net +3V3 is gone; now on net +3.3V: J5.13, J5.7, J5.8
- net +5v is gone; now on net +5V: Module1.77 (+5v_(Input)), Module1.79 (+5v_(Input)), Module1.81 (+5v_(Input)), Module1.83 (+5v_(Input)), Module1.85 (+5v_(Input)), Module1.87 (+5v_(Input))
- net EEPROM_nWP is gone; now on net GND: Module1.20 (EEPROM_nWP)
- net GPIO10 is gone; now on net GPIO_10_DB2: Module1.44 (GPIO10)
- net GPIO11 is gone; now on net GPIO_11_DB3: Module1.38 (GPIO11)
- net GPIO12 is gone; now on net GPIO_12_DB4: Module1.31 (GPIO12)
- net GPIO13 is gone; now on net GPIO_13_DB5: Module1.28 (GPIO13)
- net GPIO14 is gone; now on net GPIO_14_DB6: Module1.55 (GPIO14)
- net GPIO15 is gone; now on net GPIO_15_DB7: Module1.51 (GPIO15)
- net GPIO16 is gone; now on net GPIO_16_DB8: Module1.29 (GPIO16)
- net GPIO17 is gone; now on net GPIO_17_DB9: Module1.50 (GPIO17)
- net GPIO18 is gone; now on net GPIO_18_DB10: Module1.49 (GPIO18)
- net GPIO19 is gone; now on net GPIO_19_DB11: Module1.26 (GPIO19)
- net GPIO2 is gone; now on net GPIO_02_USB_!RESET: Module1.58 (GPIO2)
- net GPIO20 is gone; now on net GPIO_20_DB12: Module1.27 (GPIO20)
- net GPIO21 is gone; now on net GPIO_21_DB13: Module1.25 (GPIO21)
- net GPIO22 is gone; now on net GPIO_22_DB14: Module1.46 (GPIO22)
- net GPIO23 is gone; now on net GPIO_23_DB15: Module1.47 (GPIO23)
- net GPIO25 is gone; now on net GPIO_25_PWM: Module1.41 (GPIO25)
- net GPIO26 is gone; now on net GPIO_26_DAT_CMD: Module1.24 (GPIO26)
- net GPIO27 is gone; now on net GPIO_27_!RESET: Module1.48 (GPIO27)
- net GPIO7 is gone; now on net GPIO_07_!WRITE: Module1.37 (GPIO7)
- net GPIO8 is gone; now on net GPIO_08_DB0: Module1.39 (GPIO8)
- net GPIO9 is gone; now on net GPIO_09_DB1: Module1.40 (GPIO9)
- net SYNC_IN is gone; now on net GND: Module1.16 (Ethernet_SYNC_IN(1.8v))
- net SYNC_OUT is gone; now on net GND: Module1.18 (Ethernet_SYNC_OUT(1.8v))
- net TRD0_N is gone; now on net GND: Module1.10 (Ethernet_Pair0_N)
- net TRD1_N is gone; now on net GND: Module1.6 (Ethernet_Pair1_N)
- net TRD1_P is gone; now on net GND: Module1.4 (Ethernet_Pair1_P)
- net +3.3V: now also C6.1, U7.8 (VCC)
- net GND: now also C6.2, U7.2 (E1), U7.3 (E2), U7.4 (VSS), U7.7 (*WC)
- net SCL0: now also U7.6 (SCL)
- net SDA0: now also U7.5 (SDA)
- net CAM_GPIO: no longer names the net of Module1.97 (Camera_GPIO)
- net Reserved: no longer names the net of Module1.76 (Reserved)
- no-connect marks 36 -> 38
Other:
- note added: "I2C NVRAM"
- note added: "SCHEMATIC TODO: [x] Choose xtal for USB hub [x] Choose caps for xtal [x] Wire up USB hub (both ends) [x] Decide on RESET line for USB hub [x] Wire up power connections [x] Figure out GPIO mappings for display [x] Choose a GPIO for USB_RESET [x] Wire up display connections [ ] Review all RPi pinouts vs. CM4IO [x] Figure out J1 footprint & pinouts [x] Add I2C NVRAM"
- note removed: "SCHEMATIC TODO: [x] Choose xtal for USB hub [x] Choose caps for xtal [x] Wire up USB hub (both ends) [x] Decide on RESET line for USB hub [x] Wire up power connections [x] Figure out GPIO mappings for display [x] Choose a GPIO for USB_RESET [ ] Wire up display connections [ ] Review all RPi pinouts vs. CM4IO [x] Figure out J1 footprint & pinouts"
- moved on the sheet: Module1A, TP11, TP12

Commit message: Routing the board.
Connections:
- net GND: no longer Module1.10 (Ethernet_Pair0_N), Module1.16 (Ethernet_SYNC_IN(1.8v)), Module1.18 (Ethernet_SYNC_OUT(1.8v)), Module1.20 (EEPROM_nWP), Module1.4 (Ethernet_Pair1_P), Module1.6 (Ethernet_Pair1_N)
- net TRD0_P: no longer names the net of Module1.12 (Ethernet_Pair0_P)

Commit message: First complete routing done.
Connections:
- net +3.3v is gone; now on net +3.3V: D1.2 (A), D2.2 (A), Module1.78 (GPIO_VREF(1.8v/3.3v_Input)), Module1.84 (+3.3v_(Output)), Module1.86 (+3.3v_(Output)), R3.1, U2.5 (VCC), U3.5 (IN)
- net nPWR_LED: now also Module1.95 (nPI_LED_PWR)
- net +1.8v renamed +1.8V
Changed lines of the file:
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@@
     (stroke (width 0) (type solid) (color 0 0 0 0))
+  )
+  (wire (pts (xy 287.655 172.085) (xy 293.37 172.085))
+    (stroke (width 0) (type default) (color 0 0 0 0))
   )
   (wire (pts (xy 287.655 133.985) (xy 288.925 133.985))
@@
     (effects (font (size 1.27 1.27)) (justify left bottom))
   )
-  (label "+3.3v" (at 429.895 110.49 180)
+  (label "+3.3V" (at 429.895 110.49 180)
     (effects (font (size 1.27 1.27)) (justify right bottom))
   )
@@
     (effects (font (size 1.27 1.27)) (justify left bottom))
   )
-  (label "+3.3v" (at 467.36 110.49 180)
+  (label "+3.3V" (at 467.36 110.49 180)
     (effects (font (size 1.27 1.27)) (justify right bottom))
   )
@@
     (effects (font (size 1.27 1.27)) (justify left bottom))
   )
-  (label "+3.3v" (at 462.915 79.375 180)
+  (label "+3.3V" (at 462.915 79.375 180)
     (effects (font (size 1.27 1.27)) (justify right bottom))
   )
@@
     (effects (font (size 1.27 1.27)) (justify left bottom))
   )
-  (label "+3.3v" (at 455.93 127 180)
+  (label "+3.3V" (at 455.93 127 180)
     (effects (font (size 1.27 1.27)) (justify right bottom))
   )
@@
     (effects (font (size 1.27 1.27)) (justify left bottom))
   )
-  (label "+3.3v" (at 514.35 109.855 180)
+  (label "+3.3V" (at 514.35 109.855 180)
     (effects (font (size 1.27 1.27)) (justify right bottom))
   )
@@
     )
   )
-  (global_label "+3.3v" (shape input) (at 220.98 156.845 180) (fields_autoplaced)
-    (effects (font (size 1.27 1.27)) (justify right))
-    (property "Intersheet References" "${INTERSHEET_REFS}" (id 0) (at 212.8126 156.7656 0)
+  (global_label "+3.3V" (shape input) (at 220.98 156.845 180) (fields_autoplaced)
+    (effects (font (size 1.27 1.27)) (justify right))
+    (property "Intersheet References" "${INTERSHEET_REFS}" (id 0) (at 212.6916 156.7656 0)
       (effects (font (size 1.27 1.27)) (justify right) hide)
     )
@@
     )
   )
+  (global_label "nPWR_LED" (shape input) (at 293.37 172.085 0) (fields_autoplaced)
+    (effects (font (size 1.27 1.27)) (justify left))
+    (property "Intersheet References" "${INTERSHEET_REFS}" (id 0) (at 305.5288 172.0056 0)
+      (effects (font (size 1.27 1.27)) (justify left) hide)
+    )
+  )
   (global_label "CAM1_D3_P" (shape input) (at 139.7 104.775 0) (fields_autoplaced)
     (effects (font (size 1.27 1.27)) (justify left))
@@
     )
   )
-  (global_label "+1.8v" (shape input) (at 220.98 161.925 180) (fields_autoplaced)
-    (effects (font (size 1.27 1.27)) (justify right))
-    (property "Intersheet References" "${INTERSHEET_REFS}" (id 0) (at 212.8126 161.8456 0)
-      (effects (font (size 1.27 1.27)) (justify right) hide)
-    )
+  (global_label "+1.8V" (shape input) (at 220.98 161.925 180) (fields_autoplaced)
+    (effects (font (size 1.27 1.27)) (justify right))
+    (property "Intersheet References" "${INTERSHEET_REFS}" (id 0) (at 212.6916 161.8456 0)
+      (effects (font (size 1.27 1.27)) (justify right) hide)
+    )

Commit message: More or less complete except for DRC.
Parts:
- added R10: 10k, Resistor_SMD:R_0402_1005Metric, symbol Device:R
- added TP13: TestPoint, TestPoint:TestPoint_Pad_D1.0mm, symbol Connector:TestPoint
Connections:
- net USBOTG_ID is gone; now on net GND: Module1.101 (USB_OTG_ID)
- net +3.3V: now also R10.1, TP13.1
- net GND: no longer Module1.33 (GND)
- net nRPIBOOT: now reaches Module1.93 (nRPIBOOT)
- net nRPIBOOT: now also R10.2
- net AIN0: no longer names the net of Module1.96 (AnalogIP0)
- net AIN1: no longer names the net of Module1.94 (AnalogIP1)
- net CAM0_C_N: no longer names the net of Module1.140 (CAM0_C_N)
- net CAM0_C_P: no longer names the net of Module1.142 (CAM0_C_P)
- net CAM0_D0_N: no longer names the net of Module1.128 (CAM0_D0_N)
- net CAM0_D0_P: no longer names the net of Module1.130 (CAM0_D0_P)
- net CAM0_D1_N: no longer names the net of Module1.134 (CAM0_D1_N)
- net CAM0_D1_P: no longer names the net of Module1.136 (CAM0_D1_P)
- net CAM1_C_N: no longer names the net of Module1.127 (CAM1_C_N)
- net CAM1_C_P: no longer names the net of Module1.129 (CAM1_C_P)
- net CAM1_D0_N: no longer names the net of Module1.115 (CAM1_D0_N)
- net CAM1_D0_P: no longer names the net of Module1.117 (CAM1_D0_P)
- net CAM1_D1_N: no longer names the net of Module1.121 (CAM1_D1_N)
- net CAM1_D1_P: no longer names the net of Module1.123 (CAM1_D1_P)
- net CAM1_D2_N: no longer names the net of Module1.133 (CAM1_D2_N)
- net CAM1_D2_P: no longer names the net of Module1.135 (CAM1_D2_P)
- net CAM1_D3_N: no longer names the net of Module1.139 (CAM1_D3_N)
- net CAM1_D3_P: no longer names the net of Module1.141 (CAM1_D3_P)
- net DSI0_C_N: no longer names the net of Module1.169 (DSI0_C_N)
- net DSI0_C_P: no longer names the net of Module1.171 (DSI0_C_P)
- net DSI0_D0_N: no longer names the net of Module1.157 (DSI0_D0_N)
- net DSI0_D0_P: no longer names the net of Module1.159 (DSI0_D0_P)
- net DSI0_D1_N: no longer names the net of Module1.163 (DSI0_D1_N)
- net DSI0_D1_P: no longer names the net of Module1.165 (DSI0_D1_P)
- net DSI1_C_N: no longer names the net of Module1.187 (DSI1_C_N)
- net DSI1_C_P: no longer names the net of Module1.189 (DSI1_C_P)
- net DSI1_D0_N: no longer names the net of Module1.175 (DSI1_D0_N)
- net DSI1_D0_P: no longer names the net of Module1.177 (DSI1_D0_P)
- net DSI1_D1_N: no longer names the net of Module1.181 (DSI1_D1_N)
- net DSI1_D1_P: no longer names the net of Module1.183 (DSI1_D1_P)
- net DSI1_D2_N: no longer names the net of Module1.193 (DSI1_D2_N)
- net DSI1_D2_P: no longer names the net of Module1.195 (DSI1_D2_P)
- net DSI1_D3_N: no longer names the net of Module1.194 (DSI1_D3_N)
- net DSI1_D3_P: no longer names the net of Module1.196 (DSI1_D3_P)
- net ETH_LEDG: no longer names the net of Module1.17 (Ethernet_nLED2(3.3v))
- net ETH_LEDY: no longer names the net of Module1.15 (Ethernet_nLED3(3.3v))
- net GPIO24: no longer names the net of Module1.45 (GPIO24)
- net GPIO3: no longer names the net of Module1.56 (GPIO3)
- net GPIO4: no longer names the net of Module1.54 (GPIO4)
- net GPIO5: no longer names the net of Module1.34 (GPIO5)
- net GPIO6: no longer names the net of Module1.30 (GPIO6)
- net HDMI0_CEC: no longer names the net of Module1.151 (HDMI0_CEC)
- net HDMI0_CK_N: no longer names the net of Module1.190 (HDMI0_CLK_N)
- net HDMI0_CK_P: no longer names the net of Module1.188 (HDMI0_CLK_P)
- net HDMI0_D0_N: no longer names the net of Module1.184 (HDMI0_TX0_N)
- net HDMI0_D0_P: no longer names the net of Module1.182 (HDMI0_TX0_P)
- net HDMI0_D1_N: no longer names the net of Module1.178 (HDMI0_TX1_N)
- net HDMI0_D1_P: no longer names the net of Module1.176 (HDMI0_TX1_P)
- net HDMI0_D2_N: no longer names the net of Module1.172 (HDMI0_TX2_N)
- net HDMI0_D2_P: no longer names the net of Module1.170 (HDMI0_TX2_P)
- net HDMI0_HOTPLUG: no longer names the net of Module1.153 (HDMI0_HOTPLUG)
- net HDMI0_SCL: no longer names the net of Module1.200 (HDMI0_SCL)
- net HDMI0_SDA: no longer names the net of Module1.199 (HDMI0_SDA)
- net HDMI1_CEC: no longer names the net of Module1.149 (HDMI1_CEC)
- net HDMI1_CK_N: no longer names the net of Module1.166 (HDMI1_CLK_N)
- net HDMI1_CK_P: no longer names the net of Module1.164 (HDMI1_CLK_P)
- net HDMI1_D0_N: no longer names the net of Module1.160 (HDMI1_TX0_N)
- net HDMI1_D0_P: no longer names the net of Module1.158 (HDMI1_TX0_P)
- net HDMI1_D1_N: no longer names the net of Module1.154 (HDMI1_TX1_N)
- net HDMI1_D1_P: no longer names the net of Module1.152 (HDMI1_TX1_P)
- net HDMI1_D2_N: no longer names the net of Module1.148 (HDMI1_TX2_N)
- net HDMI1_D2_P: no longer names the net of Module1.146 (HDMI1_TX2_P)
- net HDMI1_HOTPLUG: no longer names the net of Module1.143 (HDMI1_HOTPLUG)
- net HDMI1_SCL: no longer names the net of Module1.147 (HDMI1_SCL)
- net HDMI1_SDA: no longer names the net of Module1.145 (HDMI1_SDA)
- net ID_SC: no longer names the net of Module1.35 (ID_SC)
- net ID_SD: no longer names the net of Module1.36 (ID_SD)
- net PCIE_CLK_N: no longer names the net of Module1.112 (PCIe_CLK_N)
- net PCIE_CLK_P: no longer names the net of Module1.110 (PCIe_CLK_P)
- net PCIE_CLK_nREQ: no longer names the net of Module1.102 (PCIe_CLK_nREQ)
- net PCIE_RX_N: no longer names the net of Module1.118 (PCIe_RX_N)
- net PCIE_RX_P: no longer names the net of Module1.116 (PCIe_RX_P)
- net PCIE_TX_N: no longer names the net of Module1.124 (PCIe_TX_N)
- net PCIE_TX_P: no longer names the net of Module1.122 (PCIe_TX_P)
- net PCIE_nRST: no longer names the net of Module1.109 (PCIe_nRST)
- net RUN_PG: no longer names the net of Module1.92 (RUN_PG)
- net TRD2_N: no longer names the net of Module1.9 (Ethernet_Pair2_N)
- net TRD2_P: no longer names the net of Module1.11 (Ethernet_Pair2_P)
- net TRD3_N: no longer names the net of Module1.5 (Ethernet_Pair3_N)
- net TRD3_P: no longer names the net of Module1.3 (Ethernet_Pair3_P)
- net TV_OUT: no longer names the net of Module1.111 (VDAC_COMP)
- no-connect marks 38 -> 121
Other:
- note added: "Note GPIO_VREF pulled to +3.3V"
- note added: "Note USB_OTG_ID pulled to GND selects USB host mode."
- note removed: "GPIO voltage select"
